File: USBcanRS485.sch (KiCad schematic (older format))
At the start: 30 parts

Commit message: Выполнена трассировка
Осталось соединить полигоны
Parts:
- removed R10: 20 кОм, MOTOR_RLC:Резистор_SMD_0,063_(0603), symbol MOTOR:Резистор_0,125Вт
- removed XP2: Вилка_СНП346-5ВП21-1-В, symbol MOTOR:Вилка_СНП346-5ВП21-1-В
- added XP2: Вилка_СНП346-6ВП21-1-В, N_X:Вилка_PLD6_вертикальная, symbol MOTOR:Вилка_СНП346-6ВП21-1-В
- added XP6: Вилка_СНП346-4ВП21-1-В, Connectors:USB_B, symbol MOTOR:Вилка_СНП346-4ВП21-1-В
- C1, C2, C3, C4, C5, C6: footprint (none) -> N_RLC:Конденсатор_SMD_0603
- DD1: footprint (none) -> N_DD:Микросхема_1986ВЕ92QL
- DD2, DD3: footprint (none) -> MOTOR_DD:Микросхема_5559ИНхх
- G1: footprint (none) -> TO_SOT_Packages_SMD:SOT-89-3_Handsoldering
- HL1, HL2: footprint OTSTOINIK:Светодиод_3мм -> N_VD_HL:Светодиод_SMD_0603
- R1, R11, R2, R3, R4, R5, R6, R7, R8, R9: footprint MOTOR_RLC:Резистор_SMD_0,063_(0603) -> N_RLC:Конденсатор_SMD_0603
- VD1: footprint (none) -> TO_SOT_Packages_SMD:SOT-23-6_Handsoldering
- XP1: footprint (none) -> N_X:USB_PLUG
- XP3, XP4: footprint (none) -> N_X:Вилка_PLS8_вертикальная
- XP5: footprint (none) -> N_X:Вилка_PLS6_вертикальная
- ZQ1: footprint (none) -> N_RLC:Резонатор_РК456МДУ(DIP)
Connections:
- wire segments 70 -> 68
Other:
- note added: "USB-B"

Commit message: Проект почти закончен
Осталось добавить предохранители на вход и выход
Parts:
- added C7, C8: 16В-10мкФ, MOTOR_RLC:Конденсатор_SMD(0805), symbol MOTOR:Конденсатор_керамический
- added HL3, HL4: Светодиод, N_VD_HL:Светодиод_SMD_0603, symbol MOTOR:Светодиод
- added R10: 20 кОм, MOTOR_RLC:Конденсатор_SMD_К10-83(0603), symbol MOTOR:Резистор_0,125Вт
- added R12, R13: 15 Ом, N_RLC:Конденсатор_SMD_0603, symbol MOTOR:Резистор_0,125Вт
- added XP7: Вилка_СНП346-3ВП21-1-В, MOTOR_X:Вилка_СНП346-3ВП21-1-В, symbol MOTOR:Вилка_СНП346-3ВП21-1-В
- DD2: value 5559ИН28У -> 5559ИН10; footprint MOTOR_DD:Микросхема_5559ИНхх -> MOTOR_IMPORT_OTK:SO-8_RS485_CAN_Milandr_OTK
- DD3: footprint MOTOR_DD:Микросхема_5559ИНхх -> MOTOR_IMPORT_OTK:SO-8_RS485_CAN_Milandr_OTK
- XP5: footprint N_X:Вилка_PLS6_вертикальная -> Connector_Dsub:DSUB-9_Female_Horizontal_P2.77x2.84mm_EdgePinOffset7.70mm_Housed_MountingHolesOffset9.12mm
Connections:
- net labels added: Osc+, Osc-
- wire segments 68 -> 87
Other:
- note added: "Действительно,\nна всякий случай"
- note added: "Подтяжка к GND\nв состоянии выкл."
- note added: "Стабилизация CPU"

Commit message: Доработка проекта
Плата приведена к размерам корпуса G403. Добавлены предохранители.
Привязаны актуальные 3D-модели.
Parts:
- added FU1, FU2: Предохранитель, N_VD_HL:Fuse_1812, symbol elements:Предохранитель
Changed lines of the file:
@@
 Wire Wire Line
 	3950 4700 5100 4700
+$Comp
+L elements:Предохранитель FU1
+U 1 1 5C3D9BF8
+P 2550 1000
+F 0 "FU1" H 2550 1262 60  0000 C CNN
+F 1 "Предохранитель" H 2550 1156 60  0000 C CNN
+F 2 "N_VD_HL:Fuse_1812" H 2550 1000 60  0001 C CNN
+F 3 "" H 2550 1000 60  0001 C CNN
+	1    2550 1000
+	1    0    0    -1
+$EndComp
+Text GLabel 2150 1000 0    50   Input ~ 0
+5В
+Text GLabel 2950 1000 2    50   Input ~ 0
+GND
+$Comp
+L elements:Предохранитель FU2
+U 1 1 5C3DA1B2
+P 3850 1000
+F 0 "FU2" H 3850 1262 60  0000 C CNN
+F 1 "Предохранитель" H 3850 1156 60  0000 C CNN
+F 2 "N_VD_HL:Fuse_1812" H 3850 1000 60  0001 C CNN
+F 3 "" H 3850 1000 60  0001 C CNN
+	1    3850 1000
+	1    0    0    -1
+$EndComp
+Text GLabel 3450 1000 0    50   Input ~ 0
+5В
+Text GLabel 4250 1000 2    50   Input ~ 0
+GND
 $EndSCHEMATC
